File: KiCad/MicoBot1/MicoBot1.sch (KiCad schematic (older format))
At the start: 21 parts, among them J1 +5v, J2 Bat, J3 Motor2, J4 Motor1, J5 GND, J6 ANin, J7 Din, J8 Serial, SW1 Rst, SW2 On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

Commit message: 
Parts:
- C1: value C -> 100n
- C2, C3: value C -> 22p
- J6: value ANin -> ANALOG
- J7: value Din -> DIGITAL
- R1: value R -> 330
- R2: value R -> 10k
- Y1: value Crystal -> 16Mhz
Connections:
- net VCC: now also R2.1; no longer R2.2
- net at C1.1, SW1.1, U1.1 (~RESET~/PC6): now also R2.2
- net at C1.2, J8.6 (Pin_6): no longer R2.1
Other:
- moved on the sheet: R2
Changed lines of the file:
@@
 P 5350 4800
 F 0 "C1" H 5465 4846 50  0000 L CNN
-F 1 "C" H 5465 4755 50  0000 L CNN
+F 1 "100n" H 5465 4755 50  0000 L CNN
 F 2 "Capacitor_THT:C_Disc_D4.3mm_W1.9mm_P5.00mm" H 5388 4650 50  0001 C CNN
 F 3 "~" H 5350 4800 50  0001 C CNN
@@
 P 5850 2750
 F 0 "R1" H 5920 2796 50  0000 L CNN
-F 1 "R" H 5920 2705 50  0000 L CNN
+F 1 "330" H 5920 2705 50  0000 L CNN
 F 2 "Resistor_THT:R_Axial_DIN0204_L3.6mm_D1.6mm_P5.08mm_Horizontal" V 5780 2750 50  0001 C CNN
 F 3 "~" H 5850 2750 50  0001 C CNN
@@
 P 5450 2550
 F 0 "Y1" H 5450 2775 50  0000 C CNN
-F 1 "Crystal" H 5450 2684 50  0000 C CNN
+F 1 "16Mhz" H 5450 2684 50  0000 C CNN
 F 2 "Crystal:Crystal_HC49-4H_Vertical" H 5450 2550 50  0001 C CNN
 F 3 "~" H 5450 2550 50  0001 C CNN
@@
 P 5350 2650
 F 0 "C2" H 5442 2696 50  0000 L CNN
-F 1 "C" H 5442 2605 50  0000 L CNN
+F 1 "22p" H 5442 2605 50  0000 L CNN
 F 2 "Capacitor_THT:C_Disc_D4.3mm_W1.9mm_P5.00mm" H 5350 2650 50  0001 C CNN
 F 3 "~" H 5350 2650 50  0001 C CNN
@@
 P 5550 2650
 F 0 "C3" H 5642 2696 50  0000 L CNN
-F 1 "C" H 5642 2605 50  0000 L CNN
+F 1 "22p" H 5642 2605 50  0000 L CNN
 F 2 "Capacitor_THT:C_Disc_D4.3mm_W1.9mm_P5.00mm" H 5550 2650 50  0001 C CNN
 F 3 "~" H 5550 2650 50  0001 C CNN
@@
 L Device:R R2
 U 1 1 5D4A63EF
-P 5350 5200
-F 0 "R2" H 5420 5246 50  0000 L CNN
-F 1 "R" H 5420 5155 50  0000 L CNN
-F 2 "Resistor_THT:R_Axial_DIN0204_L3.6mm_D1.6mm_P5.08mm_Horizontal" V 5280 5200 50  0001 C CNN
-F 3 "~" H 5350 5200 50  0001 C CNN
-	1    5350 5200
+P 4850 4600
+F 0 "R2" H 4920 4646 50  0000 L CNN
+F 1 "10k" H 4920 4555 50  0000 L CNN
+F 2 "Resistor_THT:R_Axial_DIN0204_L3.6mm_D1.6mm_P5.08mm_Horizontal" V 4780 4600 50  0001 C CNN
+F 3 "~" H 4850 4600 50  0001 C CNN
+	1    4850 4600
 	1    0    0    -1
 $EndComp
 Wire Wire Line
 	4150 3250 4600 3250
-Wire Wire Line
-	5350 4950 5350 5000
-Wire Wire Line
-	5350 5000 5600 5000
-Wire Wire Line
-	5600 5000 5600 5550
-Connection ~ 5350 5000
-Wire Wire Line
-	5350 5000 5350 5050
 $Comp
 L power:VCC #PWR014
 U 1 1 5D4B6E93
-P 5150 5350
-F 0 "#PWR014" H 5150 5200 50  0001 C CNN
-F 1 "VCC" H 5167 5523 50  0000 C CNN
-F 2 "" H 5150 5350 50  0001 C CNN
-F 3 "" H 5150 5350 50  0001 C CNN
-	1    5150 5350
-	1    0    0    -1
-$EndComp
-Wire Wire Line
-	5150 5350 5150 5450
-Wire Wire Line
-	5150 5450 5350 5450
-Wire Wire Line
-	5350 5450 5350 5350
+P 4850 4450
+F 0 "#PWR014" H 4850 4300 50  0001 C CNN
+F 1 "VCC" H 4867 4623 50  0000 C CNN
+F 2 "" H 4850 4450 50  0001 C CNN
+F 3 "" H 4850 4450 50  0001 C CNN
+	1    4850 4450
+	1    0    0    -1
+$EndComp
 Wire Wire Line
 	8600 5250 8600 5350
@@
 P 5100 3450
 F 0 "J7" H 5072 3474 50  0000 R CNN
-F 1 "Din" H 5072 3383 50  0000 R CNN
+F 1 "DIGITAL" H 5072 3383 50  0000 R CNN
 F 2 "Connector_PinHeader_2.54mm:PinHeader_1x03_P2.54mm_Vertical" H 5100 3450 50  0001 C CNN
 F 3 "~" H 5100 3450 50  0001 C CNN
@@
 P 5100 2850
 F 0 "J6" H 5072 2824 50  0000 R CNN
-F 1 "ANin" H 5072 2733 50  0000 R CNN
+F 1 "ANALOG" H 5072 2733 50  0000 R CNN
 F 2 "Connector_PinHeader_2.54mm:PinHeader_1x06_P2.54mm_Vertical" H 5100 2850 50  0001 C CNN
 F 3 "~" H 5100 2850 50  0001 C CNN
@@
 Wire Wire Line
 	4000 5450 4000 5700
+Wire Wire Line
+	5350 4950 5350 5050
+Wire Wire Line
+	5350 5050 5600 5050
+Wire Wire Line
+	5600 5050 5600 5550
+Wire Wire Line
+	4850 4750 4850 4900
+Wire Wire Line
+	4850 4900 5100 4900
+Wire Wire Line
+	5100 4900 5100 4400
+Wire Wire Line
+	5100 4400 5350 4400
 $EndSCHEMATC
