File: KiCad/MicoBot1/MicoBot1.kicad_pcb (KiCad board)
At the start: 2 copper layers, 50 x 50 mm, 23 parts, among them J1 +5v, J2 Bat, J3 Motor2, J4 Motor1, J5 GND, J6 ANALOG, J7 DIGITAL, J8 Serial, SW1 Rst, SW2 On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

Commit message: 
Parts:
- added C5: 100n, Capacitor_SMD:C_1206_3216Metric, B.Cu at (113.0, 123.2)
- renumbered J5 to Gnd1, J4 to M1, J3 to M2, J1 to Vcc1
Other:
- board text added: "Bat+"
- board text added: "Bat-"
