File: KiCad/MicoBot2/MicoBot2.sch (KiCad schematic (older format))
At the start: 22 parts, among them J2 Bat, J6 ANALOG, J7 DIGITAL, J8 Serial, M1 Motor1, M2 Motor2, SW1 Rst, SW2 On, U101 ATmega328P-AU, U2 L293D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

Commit message: 
Parts:
- C1, C2, C3: footprint Capacitor_THT:C_Disc_D4.3mm_W1.9mm_P5.00mm -> Capacitor_SMD:C_1206_3216Metric
- D1: footprint LED_THT:LED_D3.0mm -> LED_SMD:LED_1206_3216Metric
- R1, R2: footprint Resistor_THT:R_Axial_DIN0204_L3.6mm_D1.6mm_P5.08mm_Horizontal -> Resistor_SMD:R_1206_3216Metric
- SW1: footprint MiLib:Pulsador_Cuadrado_6 -> Button_Switch_SMD:SW_SPST_CK_RS282G05A3
- U2: footprint Package_DIP:DIP-16_W7.62mm -> Package_SO:SOIC-16W_7.5x12.8mm_P1.27mm
Changed lines of the file:
@@
 F 0 "C1" H 5465 4846 50  0000 L CNN
 F 1 "100n" H 5465 4755 50  0000 L CNN
-F 2 "Capacitor_THT:C_Disc_D4.3mm_W1.9mm_P5.00mm" H 5388 4650 50  0001 C CNN
+F 2 "Capacitor_SMD:C_1206_3216Metric" H 5388 4650 50  0001 C CNN
 F 3 "~" H 5350 4800 50  0001 C CNN
 	1    5350 4800
@@
 F 0 "U2" H 7600 3831 50  0000 C CNN
 F 1 "L293D" H 7600 3740 50  0000 C CNN
-F 2 "Package_DIP:DIP-16_W7.62mm" H 7850 1900 50  0001 L CNN
+F 2 "Package_SO:SOIC-16W_7.5x12.8mm_P1.27mm" H 7850 1900 50  0001 L CNN
 F 3 "http://www.ti.com/lit/ds/symlink/l293.pdf" H 7300 3350 50  0001 C CNN
 	1    7600 2650
@@
 F 0 "SW1" H 6100 4685 50  0000 C CNN
 F 1 "Rst" H 6100 4594 50  0000 C CNN
-F 2 "MiLib:Pulsador_Cuadrado_6" H 6100 4600 50  0001 C CNN
+F 2 "Button_Switch_SMD:SW_SPST_CK_RS282G05A3" H 6100 4600 50  0001 C CNN
 F 3 "~" H 6100 4600 50  0001 C CNN
 	1    6100 4400
@@
 F 0 "D1" V 5889 2333 50  0000 R CNN
 F 1 "LED" V 5798 2333 50  0000 R CNN
-F 2 "LED_THT:LED_D3.0mm" H 5850 2450 50  0001 C CNN
+F 2 "LED_SMD:LED_1206_3216Metric" H 5850 2450 50  0001 C CNN
 F 3 "~" H 5850 2450 50  0001 C CNN
 	1    5850 2450
@@
 F 0 "R1" H 5920 2796 50  0000 L CNN
 F 1 "330" H 5920 2705 50  0000 L CNN
-F 2 "Resistor_THT:R_Axial_DIN0204_L3.6mm_D1.6mm_P5.08mm_Horizontal" V 5780 2750 50  0001 C CNN
+F 2 "Resistor_SMD:R_1206_3216Metric" V 5780 2750 50  0001 C CNN
 F 3 "~" H 5850 2750 50  0001 C CNN
 	1    5850 2750
@@
 F 0 "C2" H 5442 2696 50  0000 L CNN
 F 1 "22p" H 5442 2605 50  0000 L CNN
-F 2 "Capacitor_THT:C_Disc_D4.3mm_W1.9mm_P5.00mm" H 5350 2650 50  0001 C CNN
+F 2 "Capacitor_SMD:C_1206_3216Metric" H 5350 2650 50  0001 C CNN
 F 3 "~" H 5350 2650 50  0001 C CNN
 	1    5350 2650
@@
 F 0 "C3" H 5642 2696 50  0000 L CNN
 F 1 "22p" H 5642 2605 50  0000 L CNN
-F 2 "Capacitor_THT:C_Disc_D4.3mm_W1.9mm_P5.00mm" H 5550 2650 50  0001 C CNN
+F 2 "Capacitor_SMD:C_1206_3216Metric" H 5550 2650 50  0001 C CNN
 F 3 "~" H 5550 2650 50  0001 C CNN
 	1    5550 2650
@@
 F 0 "R2" H 4920 4646 50  0000 L CNN
 F 1 "10k" H 4920 4555 50  0000 L CNN
-F 2 "Resistor_THT:R_Axial_DIN0204_L3.6mm_D1.6mm_P5.08mm_Horizontal" V 4780 4600 50  0001 C CNN
+F 2 "Resistor_SMD:R_1206_3216Metric" V 4780 4600 50  0001 C CNN
 F 3 "~" H 4850 4600 50  0001 C CNN
 	1    4850 4600
